File: cube_circuit/LED_Cube.kicad_sch (KiCad schematic)
At the start: 17 parts, among them J1 Raspberry_Pi_4, Q1 IRLZ44N, Q2 IRLZ44N, Q3 IRLZ44N, Q4 IRLZ44N, Q5 IRLZ44N, Q6 IRLZ44N, Q7 IRLZ44N, Q8 IRLZ44N, U1 74HC595, U2 74HC595, U3 74HC595, U4 74HC595, U5 74HC595, U6 74HC595, U7 74HC595, U8 74HC595

Commit message: updated circuit design
Parts:
- added D1, D10, D11, D12, D13, D14, D15, D16, D17, D18, D19, D2, D20, D21, D22, D23, D24, D25, D26, D27, D28, D29, D3, D30, D31, D32, D33, D34, D35, D36, D37, D38, D39, D4, D40, D41, D42, D43, D44, D45, D46, D47, D48, D49, D5, D50, D51, D52, D53, D54, D55, D56, D57, D58, D59, D6, D60, D61, D62, D63, D64, D7, D8, D9: LED, symbol Device:LED
- added R1, R2, R3, R4, R5, R6, R7, R8: 100Ω, symbol Device:R
- added R10, R11, R12, R13, R14, R15, R16, R9: 10KΩ, symbol Device:R
- added RN2: 330Ω, symbol Device:R_Pack10
Connections:
- net +5V: now reaches U1.10 (~{SRCLR}), U1.16 (VCC), U2.12 (RCLK), U2.16 (VCC), U3.10 (~{SRCLR}), U3.16 (VCC), U4.10 (~{SRCLR}), U4.16 (VCC), U5.10 (~{SRCLR}), U5.16 (VCC), U6.10 (~{SRCLR}), U6.16 (VCC), U7.10 (~{SRCLR}), U7.16 (VCC), U8.10 (~{SRCLR}), U8.16 (VCC)
- net +5V: no longer J1.1 (3V3), J1.17 (3V3)
- net GND: now reaches U1.13 (~{OE}), U1.8 (GND), U2.13 (~{OE}), U2.8 (GND), U3.13 (~{OE}), U3.8 (GND), U4.13 (~{OE}), U4.8 (GND), U5.13 (~{OE}), U5.8 (GND), U6.13 (~{OE}), U6.8 (GND), U7.13 (~{OE}), U7.8 (GND), U8.13 (~{OE}), U8.8 (GND)
- net GND: now also Q1.3 (S), Q2.3 (S), Q3.3 (S), Q4.3 (S), Q5.3 (S), Q6.3 (S), Q7.3 (S), Q8.3 (S), R10.2, R11.2, R12.2, R13.2, R14.2, R15.2, R16.2, R9.2; no longer J1.14 (GND), J1.20 (GND), J1.25 (GND), J1.30 (GND), J1.34 (GND), J1.39 (GND), J1.6 (GND), J1.9 (GND)
- net at J1.29 (GPCLK1/GPIO05): now also R1.2
- net at J1.31 (GPCLK2/GPIO06): now also R2.2
- net at J1.32 (GPIO12/PWM0): now also R3.2
- net at J1.33 (GPIO13/PWM1): now also R4.2
- net at J1.35 (GPIO19/SPI1_MISO/PCM_FS): now also R6.2
- net at J1.36 (GPIO16/SPI1_~{CE2}): now also R5.2
- net at J1.38 (GPIO20/SPI1_MOSI/PCM_DIN/PWM1): now also R7.2
- net at J1.40 (GPIO21/SPI1_SCLK/PCM_DOUT): now also R8.2
- net at U7.15 (QA): now also U6.7 (QH)
- net at U7.7 (QH): now also U8.15 (QA)
- net at Q8.1 (G): now also R16.1, R8.1
- net at Q8.2 (D): now also D16.1 (K), D24.1 (K), D32.1 (K), D40.1 (K), D48.1 (K), D56.1 (K), D64.1 (K), D8.1 (K)
- net at U1.1 (QB): now also RN2.16 (R5.2)
- net at U1.15 (QA): now also RN2.12 (R9.2)
- net at U1.2 (QC): now also RN2.18 (R3.2)
- net at U1.3 (QD): now also RN2.17 (R4.2)
- net at U1.4 (QE): now also RN2.15 (R6.2)
- net at U1.5 (QF): now also RN2.14 (R7.2)
- net at U1.6 (QG): now also RN2.13 (R8.2)
- net at U4.7 (QH): now also U5.15 (QA)
- net at Q6.1 (G): now also R14.1, R6.1
- net at Q6.2 (D): now also D14.1 (K), D22.1 (K), D30.1 (K), D38.1 (K), D46.1 (K), D54.1 (K), D6.1 (K), D62.1 (K)
- net at U6.15 (QA): now also U5.7 (QH)
- net at Q3.1 (G): now also R11.1, R3.1
- net at Q3.2 (D): now also D11.1 (K), D19.1 (K), D27.1 (K), D3.1 (K), D35.1 (K), D43.1 (K), D51.1 (K), D59.1 (K)
- net at Q5.1 (G): now also R13.1, R5.1
- net at Q5.2 (D): now also D13.1 (K), D21.1 (K), D29.1 (K), D37.1 (K), D45.1 (K), D5.1 (K), D53.1 (K), D61.1 (K)
- net at Q2.1 (G): now also R10.1, R2.1
- net at Q2.2 (D): now also D10.1 (K), D18.1 (K), D2.1 (K), D26.1 (K), D34.1 (K), D42.1 (K), D50.1 (K), D58.1 (K)
- net at Q1.1 (G): now also R1.1, R9.1
- net at Q1.2 (D): now also D1.1 (K), D17.1 (K), D25.1 (K), D33.1 (K), D41.1 (K), D49.1 (K), D57.1 (K), D9.1 (K)
- net at Q7.1 (G): now also R15.1, R7.1
- net at Q7.2 (D): now also D15.1 (K), D23.1 (K), D31.1 (K), D39.1 (K), D47.1 (K), D55.1 (K), D63.1 (K), D7.1 (K)
- net at Q4.1 (G): now also R12.1, R4.1
- net at Q4.2 (D): now also D12.1 (K), D20.1 (K), D28.1 (K), D36.1 (K), D4.1 (K), D44.1 (K), D52.1 (K), D60.1 (K)
- new net: D33.2 (A), D34.2 (A), D35.2 (A), D36.2 (A), D37.2 (A), D38.2 (A), D39.2 (A), D40.2 (A), RN2.6 (R6.1)
- new net: D25.2 (A), D26.2 (A), D27.2 (A), D28.2 (A), D29.2 (A), D30.2 (A), D31.2 (A), D32.2 (A), RN2.7 (R7.1)
- new net: D10.2 (A), D11.2 (A), D12.2 (A), D13.2 (A), D14.2 (A), D15.2 (A), D16.2 (A), D9.2 (A), RN2.9 (R9.1)
- new net: J1.1 (3V3), J1.17 (3V3)
- new net: J1.14 (GND), J1.20 (GND), J1.25 (GND), J1.30 (GND), J1.34 (GND), J1.39 (GND), J1.6 (GND), J1.9 (GND)
- new net: D57.2 (A), D58.2 (A), D59.2 (A), D60.2 (A), D61.2 (A), D62.2 (A), D63.2 (A), D64.2 (A), RN2.3 (R3.1)
- new net: D41.2 (A), D42.2 (A), D43.2 (A), D44.2 (A), D45.2 (A), D46.2 (A), D47.2 (A), D48.2 (A), RN2.5 (R5.1)
- new net: D1.2 (A), D2.2 (A), D3.2 (A), D4.2 (A), D5.2 (A), D6.2 (A), D7.2 (A), D8.2 (A), RN2.10 (R10.1)
- new net: D17.2 (A), D18.2 (A), D19.2 (A), D20.2 (A), D21.2 (A), D22.2 (A), D23.2 (A), D24.2 (A), RN2.8 (R8.1)
- new net: D49.2 (A), D50.2 (A), D51.2 (A), D52.2 (A), D53.2 (A), D54.2 (A), D55.2 (A), D56.2 (A), RN2.4 (R4.1)
